Commit message: changed launch files and modified xacro

File: robots/hsrb4s.urdf.xacro (robot description, xacro)
@@ -60,5 +60,5 @@
     </xacro:hsrb_wrist>
     <xacro:hsrb_hand prefix="hand" parent="wrist_roll_link">
-        <origin xyz="0.012 0.0 0.1405" rpy="0.0 0.0 ${pi}"/>
+        <origin xyz="0.012 0.0 0.1405" rpy="0.0 0.0 3.141592653589793"/>
     </xacro:hsrb_hand>
     <gazebo>

File: urdf/common.xacro (robot description, xacro)
@@ -27,5 +27,4 @@
 <robot xmlns:xacro="http://www.ros.org/wiki.xacro">
   <xacro:arg name="implicit_damping" default="false" />
-  <xacro:property name="pi" value="3.14159265359"/>
   <xacro:macro name="hsrb_position_joint_transmission" params="joint reduction">
      <transmission name="${joint}_transmission">
