Commit message: merged meshes

File: robots/hsrb4s.obj.urdf (robot description, URDF)
Before this commit: robot hsrb, 46 links, 45 joints
Links:
- link arm_flex_link: geometry collision mesh filename=package://hsr_description/meshes/arm_v0/arm_flex.stl; visual mesh filename=package://hsr_description/meshes/arm_v0/arm_flex_light.obj
- link arm_lift_link: geometry collision mesh filename=package://hsr_description/meshes/arm_v0/shoulder.stl; visual mesh filename=package://hsr_description/meshes/arm_v0/shoulder.obj
- link arm_roll_link: geometry collision mesh filename=package://hsr_description/meshes/arm_v0/arm_roll.stl; visual mesh filename=package://hsr_description/meshes/arm_v0/arm_roll_light.obj
- link base_link: geometry collision mesh filename=package://hsr_description/meshes/base_v2/base.stl; visual mesh filename=package://hsr_description/meshes/base_v2/base_light.obj
- link base_range_sensor_link: geometry collision mesh filename=package://hsr_description/meshes/sensors/laser.stl; visual mesh filename=package://hsr_description/meshes/sensors/laser.obj
- link hand_l_distal_link: geometry collision mesh filename=package://hsr_description/meshes/hand_v0/l_distal.stl; visual mesh filename=package://hsr_description/meshes/hand_v0/l_distal.obj
- link hand_l_spring_proximal_link: geometry collision mesh filename=package://hsr_description/meshes/hand_v0/l_proximal.stl; visual mesh filename=package://hsr_description/meshes/hand_v0/l_proximal.obj
- link hand_palm_link: geometry collision mesh filename=package://hsr_description/meshes/hand_v0/palm.stl; visual mesh filename=package://hsr_description/meshes/hand_v0/palm.obj
- link hand_r_distal_link: geometry collision mesh filename=package://hsr_description/meshes/hand_v0/r_distal.stl; visual mesh filename=package://hsr_description/meshes/hand_v0/r_distal.obj
- link hand_r_spring_proximal_link: geometry collision mesh filename=package://hsr_description/meshes/hand_v0/r_proximal.stl; visual mesh filename=package://hsr_description/meshes/hand_v0/r_proximal.obj
- link head_l_stereo_camera_link: geometry visual mesh filename=package://hsr_description/meshes/sensors/head_camera.obj
- link head_pan_link: geometry collision mesh filename=package://hsr_description/meshes/head_v1/head_pan.stl; visual mesh filename=package://hsr_description/meshes/head_v1/head_pan.obj
- link head_r_stereo_camera_link: geometry visual mesh filename=package://hsr_description/meshes/sensors/head_camera.obj
- link head_rgbd_sensor_link: geometry collision mesh filename=package://hsr_description/meshes/sensors/rgbd.stl; visual mesh filename=package://hsr_description/meshes/sensors/rgbd_light.obj
- link head_tilt_link: geometry collision mesh filename=package://hsr_description/meshes/head_v1/head.stl; collision mesh filename=package://hsr_description/meshes/head_v1/tablet.stl
- link torso_lift_link: geometry collision mesh filename=package://hsr_description/meshes/torso_v0/torso.stl; visual mesh filename=package://hsr_description/meshes/torso_v0/torso_light.obj
- link wrist_flex_link: geometry collision cylinder length=0.04 radius=0.017; visual cylinder length=0.02 radius=0.017
- link wrist_roll_link: geometry collision mesh filename=package://hsr_description/meshes/wrist_v0/wrist_roll.stl; visual mesh filename=package://hsr_description/meshes/wrist_v0/wrist_roll.obj

File: robots/hsrb4s.urdf (robot description, URDF)
Before this commit: robot hsrb, 46 links, 45 joints
Links:
- link arm_flex_link: geometry collision mesh filename=package://hsr_description/meshes/arm_v0/arm_flex.stl; visual mesh filename=package://hsr_description/meshes/arm_v0/arm_flex_light.dae
- link arm_lift_link: geometry collision mesh filename=package://hsr_description/meshes/arm_v0/shoulder.stl; visual mesh filename=package://hsr_description/meshes/arm_v0/shoulder.dae
- link arm_roll_link: geometry collision mesh filename=package://hsr_description/meshes/arm_v0/arm_roll.stl; visual mesh filename=package://hsr_description/meshes/arm_v0/arm_roll_light.dae
- link base_link: geometry collision mesh filename=package://hsr_description/meshes/base_v2/base.stl; visual mesh filename=package://hsr_description/meshes/base_v2/base_light.dae
- link base_range_sensor_link: geometry collision mesh filename=package://hsr_description/meshes/sensors/laser.stl; visual mesh filename=package://hsr_description/meshes/sensors/laser.dae
- link hand_l_distal_link: geometry collision mesh filename=package://hsr_description/meshes/hand_v0/l_distal.stl; visual mesh filename=package://hsr_description/meshes/hand_v0/l_distal.stl
- link hand_l_spring_proximal_link: geometry collision mesh filename=package://hsr_description/meshes/hand_v0/l_proximal.stl; visual mesh filename=package://hsr_description/meshes/hand_v0/l_proximal.stl
- link hand_palm_link: geometry collision mesh filename=package://hsr_description/meshes/hand_v0/palm.stl; visual mesh filename=package://hsr_description/meshes/hand_v0/palm.stl
- link hand_r_distal_link: geometry collision mesh filename=package://hsr_description/meshes/hand_v0/r_distal.stl; visual mesh filename=package://hsr_description/meshes/hand_v0/r_distal.stl
- link hand_r_spring_proximal_link: geometry collision mesh filename=package://hsr_description/meshes/hand_v0/r_proximal.stl; visual mesh filename=package://hsr_description/meshes/hand_v0/r_proximal.stl
- link head_l_stereo_camera_link: geometry visual mesh filename=package://hsr_description/meshes/sensors/head_camera.dae
- link head_pan_link: geometry collision mesh filename=package://hsr_description/meshes/head_v1/head_pan.stl; visual mesh filename=package://hsr_description/meshes/head_v1/head_pan.dae
- link head_r_stereo_camera_link: geometry visual mesh filename=package://hsr_description/meshes/sensors/head_camera.dae
- link head_rgbd_sensor_link: geometry collision mesh filename=package://hsr_description/meshes/sensors/rgbd.stl; visual mesh filename=package://hsr_description/meshes/sensors/rgbd_light.dae
- link head_tilt_link: geometry collision mesh filename=package://hsr_description/meshes/head_v1/head.stl; collision mesh filename=package://hsr_description/meshes/head_v1/tablet.stl
- link torso_lift_link: geometry collision mesh filename=package://hsr_description/meshes/torso_v0/torso.stl; visual mesh filename=package://hsr_description/meshes/torso_v0/torso_light.dae
- link wrist_flex_link: geometry collision cylinder length=0.04 radius=0.017; visual cylinder length=0.02 radius=0.017
- link wrist_roll_link: geometry collision mesh filename=package://hsr_description/meshes/wrist_v0/wrist_roll.stl; visual mesh filename=package://hsr_description/meshes/wrist_v0/wrist_roll.dae

File: urdf/arm_v0/arm.urdf.xacro (robot description, xacro)
@@ -50,8 +50,8 @@
                 <geometry>
                     <xacro:unless value="${g_use_obj_for_visual}">
-                        <mesh filename="package://hsr_meshes/meshes/arm_v0/shoulder.dae" />
+                        <mesh filename="package://hsr_description/meshes/arm_v0/shoulder.dae" />
                     </xacro:unless>
                     <xacro:if value="${g_use_obj_for_visual}">
-                        <mesh filename="package://hsr_meshes/meshes/arm_v0/shoulder.obj" />
+                        <mesh filename="package://hsr_description/meshes/arm_v0/shoulder.obj" />
                     </xacro:if>
                 </geometry>
@@ -59,5 +59,5 @@
             <collision>
                 <geometry>
-                    <mesh filename="package://hsr_meshes/meshes/arm_v0/shoulder.stl" />
+                    <mesh filename="package://hsr_description/meshes/arm_v0/shoulder.stl" />
                 </geometry>
             </collision>
@@ -83,8 +83,8 @@
                 <geometry>
                     <xacro:unless value="${g_use_obj_for_visual}">
-                        <mesh filename="package://hsr_meshes/meshes/arm_v0/arm_flex_light.dae" />
+                        <mesh filename="package://hsr_description/meshes/arm_v0/arm_flex_light.dae" />
                     </xacro:unless>
                     <xacro:if value="${g_use_obj_for_visual}">
-                        <mesh filename="package://hsr_meshes/meshes/arm_v0/arm_flex_light.obj" />
+                        <mesh filename="package://hsr_description/meshes/arm_v0/arm_flex_light.obj" />
                     </xacro:if>
                 </geometry>
@@ -92,5 +92,5 @@
             <collision>
                 <geometry>
-                    <mesh filename="package://hsr_meshes/meshes/arm_v0/arm_flex.stl" />
+                    <mesh filename="package://hsr_description/meshes/arm_v0/arm_flex.stl" />
                 </geometry>
             </collision>
@@ -116,8 +116,8 @@
                 <geometry>
                     <xacro:unless value="${g_use_obj_for_visual}">
-                        <mesh filename="package://hsr_meshes/meshes/arm_v0/arm_roll_light.dae" />
+                        <mesh filename="package://hsr_description/meshes/arm_v0/arm_roll_light.dae" />
                     </xacro:unless>
                     <xacro:if value="${g_use_obj_for_visual}">
-                        <mesh filename="package://hsr_meshes/meshes/arm_v0/arm_roll_light.obj" />
+                        <mesh filename="package://hsr_description/meshes/arm_v0/arm_roll_light.obj" />
                     </xacro:if>
                 </geometry>
@@ -125,5 +125,5 @@
             <collision>
                 <geometry>
-                    <mesh filename="package://hsr_meshes/meshes/arm_v0/arm_roll.stl" />
+                    <mesh filename="package://hsr_description/meshes/arm_v0/arm_roll.stl" />
                 </geometry>
             </collision>

File: urdf/base_v2/base.urdf.xacro (robot description, xacro)
@@ -145,8 +145,8 @@
                 <geometry>
                     <xacro:unless value="${g_use_obj_for_visual}">
-                        <mesh filename="package://hsr_meshes/meshes/base_v2/base_light.dae" />
+                        <mesh filename="package://hsr_description/meshes/base_v2/base_light.dae" />
                     </xacro:unless>
                     <xacro:if value="${g_use_obj_for_visual}">
-                        <mesh filename="package://hsr_meshes/meshes/base_v2/base_light.obj" />
+                        <mesh filename="package://hsr_description/meshes/base_v2/base_light.obj" />
                     </xacro:if>
                 </geometry>
@@ -155,8 +155,8 @@
                 <geometry>
                     <xacro:unless value="${g_use_obj_for_visual}">
-                        <mesh filename="package://hsr_meshes/meshes/base_v2/body_light.dae" />
+                        <mesh filename="package://hsr_description/meshes/base_v2/body_light.dae" />
                     </xacro:unless>
                     <xacro:if value="${g_use_obj_for_visual}">
-                        <mesh filename="package://hsr_meshes/meshes/base_v2/body_light.obj" />
+                        <mesh filename="package://hsr_description/meshes/base_v2/body_light.obj" />
                     </xacro:if>
                 </geometry>
@@ -165,8 +165,8 @@
                 <geometry>
                     <xacro:unless value="${g_use_obj_for_visual}">
-                        <mesh filename="package://hsr_meshes/meshes/base_v2/torso_base.dae" />
+                        <mesh filename="package://hsr_description/meshes/base_v2/torso_base.dae" />
                     </xacro:unless>
                     <xacro:if value="${g_use_obj_for_visual}">
-                        <mesh filename="package://hsr_meshes/meshes/base_v2/torso_base.obj" />
+                        <mesh filename="package://hsr_description/meshes/base_v2/torso_base.obj" />
                     </xacro:if>
                 </geometry>
@@ -174,5 +174,5 @@
             <collision>
                 <geometry>
-                    <mesh filename="package://hsr_meshes/meshes/base_v2/base.stl" />
+                    <mesh filename="package://hsr_description/meshes/base_v2/base.stl" />
                 </geometry>
             </collision>

File: urdf/hand_v0/hand.urdf.xacro (robot description, xacro)
@@ -66,15 +66,15 @@
                 <geometry>
                     <xacro:unless value="${g_use_obj_for_visual}">
-                        <mesh filename="package://hsr_meshes/meshes/hand_v0/palm.stl" />
-                    </xacro:unless>
-                    <xacro:if value="${g_use_obj_for_visual}">
-                        <mesh filename="package://hsr_meshes/meshes/hand_v0/palm.obj" />
-                    </xacro:if>
-                </geometry>
-                <material name="body_sub" />
-            </visual>
-            <collision>
-                <geometry>
-                    <mesh filename="package://hsr_meshes/meshes/hand_v0/palm.stl" />
+                        <mesh filename="package://hsr_description/meshes/hand_v0/palm.stl" />
+                    </xacro:unless>
+                    <xacro:if value="${g_use_obj_for_visual}">
+                        <mesh filename="package://hsr_description/meshes/hand_v0/palm.obj" />
+                    </xacro:if>
+                </geometry>
+                <material name="body_sub" />
+            </visual>
+            <collision>
+                <geometry>
+                    <mesh filename="package://hsr_description/meshes/hand_v0/palm.stl" />
                 </geometry>
             </collision>
@@ -185,15 +185,15 @@
                 <geometry>
                     <xacro:unless value="${g_use_obj_for_visual}">
-                        <mesh filename="package://hsr_meshes/meshes/hand_v0/l_proximal.stl" />
-                    </xacro:unless>
-                    <xacro:if value="${g_use_obj_for_visual}">
-                        <mesh filename="package://hsr_meshes/meshes/hand_v0/l_proximal.obj" />
-                    </xacro:if>
-                </geometry>
-                <material name="body_sub" />
-            </visual>
-            <collision>
-                <geometry>
-                    <mesh filename="package://hsr_meshes/meshes/hand_v0/l_proximal.stl" />
+                        <mesh filename="package://hsr_description/meshes/hand_v0/l_proximal.stl" />
+                    </xacro:unless>
+                    <xacro:if value="${g_use_obj_for_visual}">
+                        <mesh filename="package://hsr_description/meshes/hand_v0/l_proximal.obj" />
+                    </xacro:if>
+                </geometry>
+                <material name="body_sub" />
+            </visual>
+            <collision>
+                <geometry>
+                    <mesh filename="package://hsr_description/meshes/hand_v0/l_proximal.stl" />
                 </geometry>
             </collision>
@@ -214,15 +214,15 @@
                 <geometry>
                     <xacro:unless value="${g_use_obj_for_visual}">
-                        <mesh filename="package://hsr_meshes/meshes/hand_v0/l_distal.stl" />
-                    </xacro:unless>
-                    <xacro:if value="${g_use_obj_for_visual}">
-                        <mesh filename="package://hsr_meshes/meshes/hand_v0/l_distal.obj" />
-                    </xacro:if>
-                </geometry>
-                <material name="body_sub" />
-            </visual>
-            <collision>
-                <geometry>
-                    <mesh filename="package://hsr_meshes/meshes/hand_v0/l_distal.stl" />
+                        <mesh filename="package://hsr_description/meshes/hand_v0/l_distal.stl" />
+                    </xacro:unless>
+                    <xacro:if value="${g_use_obj_for_visual}">
+                        <mesh filename="package://hsr_description/meshes/hand_v0/l_distal.obj" />
+                    </xacro:if>
+                </geometry>
+                <material name="body_sub" />
+            </visual>
+            <collision>
+                <geometry>
+                    <mesh filename="package://hsr_description/meshes/hand_v0/l_distal.stl" />
                 </geometry>
             </collision>
@@ -273,15 +273,15 @@
                 <geometry>
                     <xacro:unless value="${g_use_obj_for_visual}">
-                        <mesh filename="package://hsr_meshes/meshes/hand_v0/r_proximal.stl" />
-                    </xacro:unless>
-                    <xacro:if value="${g_use_obj_for_visual}">
-                        <mesh filename="package://hsr_meshes/meshes/hand_v0/r_proximal.obj" />
-                    </xacro:if>
-                </geometry>
-                <material name="body_sub" />
-            </visual>
-            <collision>
-                <geometry>
-                    <mesh filename="package://hsr_meshes/meshes/hand_v0/r_proximal.stl" />
+                        <mesh filename="package://hsr_description/meshes/hand_v0/r_proximal.stl" />
+                    </xacro:unless>
+                    <xacro:if value="${g_use_obj_for_visual}">
+                        <mesh filename="package://hsr_description/meshes/hand_v0/r_proximal.obj" />
+                    </xacro:if>
+                </geometry>
+                <material name="body_sub" />
+            </visual>
+            <collision>
+                <geometry>
+                    <mesh filename="package://hsr_description/meshes/hand_v0/r_proximal.stl" />
                 </geometry>
             </collision>
@@ -302,15 +302,15 @@
                 <geometry>
                     <xacro:unless value="${g_use_obj_for_visual}">
-                        <mesh filename="package://hsr_meshes/meshes/hand_v0/r_distal.stl" />
-                    </xacro:unless>
-                    <xacro:if value="${g_use_obj_for_visual}">
-                        <mesh filename="package://hsr_meshes/meshes/hand_v0/r_distal.obj" />
-                    </xacro:if>
-                </geometry>
-                <material name="body_sub" />
-            </visual>
-            <collision>
-                <geometry>
-                    <mesh filename="package://hsr_meshes/meshes/hand_v0/r_distal.stl" />
+                        <mesh filename="package://hsr_description/meshes/hand_v0/r_distal.stl" />
+                    </xacro:unless>
+                    <xacro:if value="${g_use_obj_for_visual}">
+                        <mesh filename="package://hsr_description/meshes/hand_v0/r_distal.obj" />
+                    </xacro:if>
+                </geometry>
+                <material name="body_sub" />
+            </visual>
+            <collision>
+                <geometry>
+                    <mesh filename="package://hsr_description/meshes/hand_v0/r_distal.stl" />
                 </geometry>
             </collision>

File: urdf/head_v2/head.urdf.xacro (robot description, xacro)
@@ -53,8 +53,8 @@
                 <geometry>
                     <xacro:unless value="${g_use_obj_for_visual}">
-                        <mesh filename="package://hsr_meshes/meshes/head_v1/head_pan.dae" />
+                        <mesh filename="package://hsr_description/meshes/head_v1/head_pan.dae" />
                     </xacro:unless>
                     <xacro:if value="${g_use_obj_for_visual}">
-                        <mesh filename="package://hsr_meshes/meshes/head_v1/head_pan.obj" />
+                        <mesh filename="package://hsr_description/meshes/head_v1/head_pan.obj" />
                     </xacro:if>
                 </geometry>
@@ -62,5 +62,5 @@
             <collision>
                 <geometry>
-                    <mesh filename="package://hsr_meshes/meshes/head_v1/head_pan.stl" />
+                    <mesh filename="package://hsr_description/meshes/head_v1/head_pan.stl" />
                 </geometry>
             </collision>
@@ -86,8 +86,8 @@
                 <geometry>
                     <xacro:unless value="${g_use_obj_for_visual}">
-                        <mesh filename="package://hsr_meshes/meshes/head_v1/head_upper.dae" />
+                        <mesh filename="package://hsr_description/meshes/head_v1/head_upper.dae" />
                     </xacro:unless>
                     <xacro:if value="${g_use_obj_for_visual}">
-                        <mesh filename="package://hsr_meshes/meshes/head_v1/head_upper.obj" />
+                        <mesh filename="package://hsr_description/meshes/head_v1/head_upper.obj" />
                     </xacro:if>
                 </geometry>
@@ -96,8 +96,8 @@
                 <geometry>
                     <xacro:unless value="${g_use_obj_for_visual}">
-                        <mesh filename="package://hsr_meshes/meshes/head_v1/head_tilt.dae" />
+                        <mesh filename="package://hsr_description/meshes/head_v1/head_tilt.dae" />
                     </xacro:unless>
                     <xacro:if value="${g_use_obj_for_visual}">
-                        <mesh filename="package://hsr_meshes/meshes/head_v1/head_tilt.obj" />
+                        <mesh filename="package://hsr_description/meshes/head_v1/head_tilt.obj" />
                     </xacro:if>
                 </geometry>
@@ -106,8 +106,8 @@
                 <geometry>
                     <xacro:unless value="${g_use_obj_for_visual}">
-                        <mesh filename="package://hsr_meshes/meshes/head_v1/tablet_base.dae" />
+                        <mesh filename="package://hsr_description/meshes/head_v1/tablet_base.dae" />
                     </xacro:unless>
                     <xacro:if value="${g_use_obj_for_visual}">
-                        <mesh filename="package://hsr_meshes/meshes/head_v1/tablet_base.obj" />
+                        <mesh filename="package://hsr_description/meshes/head_v1/tablet_base.obj" />
                     </xacro:if>
                 </geometry>
@@ -115,10 +115,10 @@
             <collision>
                 <geometry>
-                    <mesh filename="package://hsr_meshes/meshes/head_v1/head.stl" />
+                    <mesh filename="package://hsr_description/meshes/head_v1/head.stl" />
                 </geometry>
             </collision>
             <collision>
                 <geometry>
-                    <mesh filename="package://hsr_meshes/meshes/head_v1/tablet.stl" />
+                    <mesh filename="package://hsr_description/meshes/head_v1/tablet.stl" />
                 </geometry>
             </collision>
