Commit message: merged meshes

File: urdf/sensors/laser.urdf.xacro (robot description, xacro)
@@ -38,8 +38,8 @@
                 <geometry>
                     <xacro:unless value="${g_use_obj_for_visual}">
-                        <mesh filename="package://hsr_meshes/meshes/sensors/laser.dae" />
+                        <mesh filename="package://hsr_description/meshes/sensors/laser.dae" />
                     </xacro:unless>
                     <xacro:if value="${g_use_obj_for_visual}">
-                        <mesh filename="package://hsr_meshes/meshes/sensors/laser.obj" />
+                        <mesh filename="package://hsr_description/meshes/sensors/laser.obj" />
                     </xacro:if>
                 </geometry>
@@ -47,5 +47,5 @@
             <collision>
                 <geometry>
-                    <mesh filename="package://hsr_meshes/meshes/sensors/laser.stl" />
+                    <mesh filename="package://hsr_description/meshes/sensors/laser.stl" />
                 </geometry>
             </collision>

File: urdf/sensors/rgb_sensor.urdf.xacro (robot description, xacro)
@@ -38,8 +38,8 @@
                 <geometry>
                     <xacro:if value="${g_use_obj_for_visual}">
-                        <mesh filename="package://hsr_meshes/meshes/sensors/head_camera.obj" />
+                        <mesh filename="package://hsr_description/meshes/sensors/head_camera.obj" />
                     </xacro:if>
                     <xacro:unless value="${g_use_obj_for_visual}">
-                        <mesh filename="package://hsr_meshes/meshes/sensors/head_camera.dae" />
+                        <mesh filename="package://hsr_description/meshes/sensors/head_camera.dae" />
                     </xacro:unless>
                 </geometry>

File: urdf/sensors/rgbd_sensor.urdf.xacro (robot description, xacro)
@@ -38,8 +38,8 @@
                 <geometry>
                     <xacro:unless value="${g_use_obj_for_visual}">
-                        <mesh filename="package://hsr_meshes/meshes/sensors/rgbd_light.dae" />
+                        <mesh filename="package://hsr_description/meshes/sensors/rgbd_light.dae" />
                     </xacro:unless>
                     <xacro:if value="${g_use_obj_for_visual}">
-                        <mesh filename="package://hsr_meshes/meshes/sensors/rgbd_light.obj" />
+                        <mesh filename="package://hsr_description/meshes/sensors/rgbd_light.obj" />
                     </xacro:if>
                 </geometry>
@@ -48,5 +48,5 @@
                 <origin xyz="0 0 0" rpy="0.0 0.0 0.0"/>
                 <geometry>
-                    <mesh filename="package://hsr_meshes/meshes/sensors/rgbd.stl" />
+                    <mesh filename="package://hsr_description/meshes/sensors/rgbd.stl" />
                 </geometry>
             </collision>

File: urdf/torso_v0/torso.urdf.xacro (robot description, xacro)
@@ -49,8 +49,8 @@
                 <geometry>
                     <xacro:unless value="${g_use_obj_for_visual}">
-                        <mesh filename="package://hsr_meshes/meshes/torso_v0/torso_light.dae" />
+                        <mesh filename="package://hsr_description/meshes/torso_v0/torso_light.dae" />
                     </xacro:unless>
                     <xacro:if value="${g_use_obj_for_visual}">
-                        <mesh filename="package://hsr_meshes/meshes/torso_v0/torso_light.obj" />
+                        <mesh filename="package://hsr_description/meshes/torso_v0/torso_light.obj" />
                     </xacro:if>
                 </geometry>
@@ -58,5 +58,5 @@
             <collision>
                 <geometry>
-                    <mesh filename="package://hsr_meshes/meshes/torso_v0/torso.stl" />
+                    <mesh filename="package://hsr_description/meshes/torso_v0/torso.stl" />
                 </geometry>
             </collision>

File: urdf/wrist_v0/wrist.urdf.xacro (robot description, xacro)
@@ -51,8 +51,8 @@
                 <geometry>
                     <xacro:unless value="${g_use_obj_for_visual}">
-                        <mesh filename="package://hsr_meshes/meshes/wrist_v0/wrist_flex.dae" />
+                        <mesh filename="package://hsr_description/meshes/wrist_v0/wrist_flex.dae" />
                     </xacro:unless>
                     <xacro:if value="${g_use_obj_for_visual}">
-                        <mesh filename="package://hsr_meshes/meshes/wrist_v0/wrist_flex.obj" />
+                        <mesh filename="package://hsr_description/meshes/wrist_v0/wrist_flex.obj" />
                     </xacro:if>
                 </geometry>
@@ -93,8 +93,8 @@
                 <geometry>
                     <xacro:unless value="${g_use_obj_for_visual}">
-                        <mesh filename="package://hsr_meshes/meshes/wrist_v0/wrist_roll.dae" />
+                        <mesh filename="package://hsr_description/meshes/wrist_v0/wrist_roll.dae" />
                     </xacro:unless>
                     <xacro:if value="${g_use_obj_for_visual}">
-                        <mesh filename="package://hsr_meshes/meshes/wrist_v0/wrist_roll.obj" />
+                        <mesh filename="package://hsr_description/meshes/wrist_v0/wrist_roll.obj" />
                     </xacro:if>
                 </geometry>
@@ -102,5 +102,5 @@
             <collision>
                 <geometry>
-                    <mesh filename="package://hsr_meshes/meshes/wrist_v0/wrist_roll.stl" />
+                    <mesh filename="package://hsr_description/meshes/wrist_v0/wrist_roll.stl" />
                 </geometry>
             </collision>
